File: Hardware/L6470 AutoDriver.sch (EAGLE design)
At the start: 39 parts, among them U1 L6470

Commit message: Final file changes from revision
Parts:
- renumbered SJ4 to SJ3
Other:
- note added: "SJ3 allows you to route the SDO (serial data out) either to the next board (if this board is in a chain) or back to the previous board (if this board is the last or only board in the chain). It defaults to back to previous board, for single board applications."
- note added: "Vs must be between 8V and 45V Motor supply must be enabled for chip comms to work!"
- note removed: "SJ4 allows you to route the SDO (serial data out) either to the next board (if this board is in a chain) or back to the previous board (if this board is the last or only board in the chain). It defaults to back to previous board, for single board applications."
- note removed: "Vs must be between 8V and 45V"
Changed lines of the file:
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@@
 <?xml version="1.0" encoding="utf-8"?>
 <!DOCTYPE eagle SYSTEM "eagle.dtd">
-<eagle version="7.3.0">
+<eagle version="7.5.0">
 <drawing>
 <settings>
@@
 <layer number="255" name="routoute" color="7" fill="1" visible="yes" active="yes"/>
 </layers>
-<schematic xreflabel="%F%N/%S" xrefpart="1_/%S.%C%R">
+<schematic xreflabel="%F%N/%S" xrefpart="/%S.%C%R">
 <attributes>
 </attributes>
@@
 <part name="TP1" library="SparkFun-Passives" deviceset="TEST-POINT" device="TP_15TH_THRU"/>
 <part name="FRAME1" library="SparkFun-Aesthetics" deviceset="FRAME-LETTER" device=""/>
-<part name="SJ4" library="SparkFun-Passives" deviceset="JUMPER-PAD-3-2OF3_NC_BY_PASTE" device=""/>
+<part name="SJ3" library="SparkFun-Passives" deviceset="JUMPER-PAD-3-2OF3_NC_BY_PASTE" device=""/>
 </parts>
 <sheets>
@@
 5 Mbit max</text>
 <wire x1="157.48" y1="147.32" x2="154.94" y2="147.32" width="0.508" layer="94"/>
-<wire x1="0" y1="40.64" x2="73.66" y2="40.64" width="0.3048" layer="97" style="longdash"/>
-<wire x1="73.66" y1="40.64" x2="73.66" y2="185.42" width="0.3048" layer="97" style="longdash"/>
+<wire x1="0" y1="53.34" x2="73.66" y2="53.34" width="0.3048" layer="97" style="longdash"/>
+<wire x1="73.66" y1="53.34" x2="73.66" y2="185.42" width="0.3048" layer="97" style="longdash"/>
 <wire x1="147.32" y1="35.56" x2="73.66" y2="35.56" width="0.3048" layer="97" style="longdash"/>
-<wire x1="73.66" y1="35.56" x2="73.66" y2="40.64" width="0.3048" layer="97" style="longdash"/>
+<wire x1="73.66" y1="35.56" x2="73.66" y2="53.34" width="0.3048" layer="97" style="longdash"/>
 <text x="172.72" y="7.62" size="2.54" layer="94">Mike Hord
 </text>
-<text x="3.048" y="37.084" size="2.54" layer="97">Vs must be between 8V and 45V</text>
+<text x="3.048" y="42.164" size="2.54" layer="97">Vs must be between 8V and 45V
+Motor supply must be enabled
+for chip comms to work!</text>
 <text x="238.76" y="7.62" size="2.54" layer="94">12</text>
-<text x="76.2" y="167.64" size="1.778" layer="97">SJ4 allows you to route the SDO (serial
+<text x="76.2" y="167.64" size="1.778" layer="97">SJ3 allows you to route the SDO (serial
 data out) either to the next board (if this
 board is in a chain) or back to the previous
@@
 <instance part="FRAME1" gate="G$1" x="0" y="0"/>
 <instance part="FRAME1" gate="V" x="147.32" y="0"/>
-<instance part="SJ4" gate="G$1" x="101.6" y="162.56" smashed="yes" rot="R90">
+<instance part="SJ3" gate="G$1" x="101.6" y="162.56" smashed="yes" rot="R90">
 <attribute name="NAME" x="99.822" y="164.465" size="1.778" layer="95"/>
 </instance>
@@
 </segment>
 <segment>
-<pinref part="SJ4" gate="G$1" pin="3"/>
+<pinref part="SJ3" gate="G$1" pin="3"/>
 <wire x1="106.68" y1="162.56" x2="109.22" y2="162.56" width="0.1524" layer="91"/>
 <label x="109.22" y="162.56" size="1.27" layer="95" xref="yes"/>
@@
 </segment>
 <segment>
-<pinref part="SJ4" gate="G$1" pin="2"/>
+<pinref part="SJ3" gate="G$1" pin="2"/>
 <wire x1="101.6" y1="157.48" x2="101.6" y2="154.94" width="0.1524" layer="91"/>
 <wire x1="101.6" y1="154.94" x2="109.22" y2="154.94" width="0.1524" layer="91"/>
@@
 </segment>
 <segment>
-<pinref part="SJ4" gate="G$1" pin="1"/>
+<pinref part="SJ3" gate="G$1" pin="1"/>
 <wire x1="96.52" y1="162.56" x2="93.98" y2="162.56" width="0.1524" layer="91"/>
 <label x="93.98" y="162.56" size="1.27" layer="95" rot="R180" xref="yes"/>
