File: Hardware/L6470 AutoDriver.brd (EAGLE design)
At the start: 73.7 x 49.5 mm, 39 parts, among them U1 L6470

Commit message: Fixed BSilk to match TSilk, advanced version number
Other:
- board text added: "v13"
- board text removed: "MISO"
- board text removed: "MOSI"
- board text removed: "v12"
Changed lines of the file:
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@@
 <text x="8.001" y="41.91" size="0.8128" layer="22" font="vector" ratio="15" rot="SMR270" align="bottom-right">GND</text>
 <text x="10.541" y="41.91" size="0.8128" layer="22" font="vector" ratio="15" rot="SMR270" align="bottom-right">OSCOUT</text>
-<text x="13.081" y="41.91" size="0.8128" layer="22" font="vector" ratio="15" rot="SMR270" align="bottom-right">MOSI</text>
-<text x="15.621" y="41.91" size="0.8128" layer="22" font="vector" ratio="15" rot="SMR270" align="bottom-right">MISO</text>
 <text x="18.161" y="41.91" size="0.8128" layer="22" font="vector" ratio="15" rot="SMR270" align="bottom-right">3-5V</text>
 <text x="28.321" y="41.91" size="0.8128" layer="22" font="vector" ratio="15" rot="SMR270" align="bottom-right">GND</text>
@@
 <text x="1.27" y="36.83" size="1.778" layer="15" font="vector" ratio="15">3</text>
 <text x="5.08" y="36.83" size="1.778" layer="16" font="vector" ratio="15" rot="MR0">4</text>
-<text x="2.54" y="35.56" size="1.778" layer="16" font="vector" ratio="15" rot="MR270">v12</text>
+<text x="2.54" y="35.56" size="1.778" layer="16" font="vector" ratio="15" rot="MR270">v13</text>
 <dimension x1="0" y1="49.53" x2="73.66" y2="49.53" x3="36.83" y3="55.88" textsize="1.778" textratio="15" layer="47" unit="inch"/>
 <dimension x1="0" y1="0" x2="0" y2="49.53" x3="-6.35" y3="24.765" textsize="1.778" textratio="15" layer="47" unit="inch"/>
@@
 <dimension x1="2.54" y1="2.54" x2="-7.62" y2="-2.54" x3="-13.97" y3="-2.54" textsize="1.778" textratio="15" layer="47" dtype="leader" unit="inch"/>
 <text x="-25.4" y="-3.81" size="1.778" layer="47" font="vector" ratio="15">M3/4-40</text>
+<text x="13.081" y="41.91" size="0.8128" layer="22" font="vector" ratio="15" rot="SMR270" align="bottom-right">SD to
+next bd</text>
+<text x="15.621" y="41.91" size="0.8128" layer="22" font="vector" ratio="15" rot="SMR270" align="bottom-right">!CS</text>
+<text x="31.496" y="41.91" size="0.8128" layer="22" font="vector" ratio="15" rot="SMR270" align="bottom-right">SD to
+prev bd</text>
 </plain>
 <attributes>
