File: Production/L6470AutoDriver-Panel_v13.brd (EAGLE design)
At the start: 309.9 x 163.3 mm, 447 parts, among them U1 L6470, U10 L6470, U11 L6470, U12 L6470, U2 L6470, U3 L6470, U4 L6470, U5 L6470, U6 L6470, U7 L6470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

Commit message: created panel v13
Parts:
- moved E$5 134.9 mm to (304.7, 14.5), turned to 0 degrees
- moved E$6 131.1 mm to (304.7, 147.1), turned to 180 degrees
- moved E$1 3.81 mm to (4.57, 10.9)
Other:
- outline, holes or cut-outs redrawn
- board text added: "This is a four layer cake board!!"
- board text added: "v13"
- board text removed: "BUSYN"
- board text removed: "MISO"
- board text removed: "MOSI"
- board text removed: "This is a 4-layer cake board!!"
- board text removed: "v12"
